File: hardware/multiplexer-1vX/design.brd (EAGLE design)
At the start: 100 x 100 mm, 64 parts, among them IC10 ISO1540D, IC9 TCA9554APWR, X1 DG3XX-02-5.0, X10 DG3XX-02-5.0, X11 DG3XX-02-5.0, X2 04-JST-B4B-XH-A, X3 DG3XX-02-5.0, X4 DG3XX-02-5.0, X5 DG3XX-02-5.0, X6 DG3XX-02-5.0, X7 DG3XX-02-5.0, X8 DG3XX-02-5.0, X9 DG3XX-02-5.0

Commit message: Update hardware
Parts:
- added C13: (no value), microbuilder:0805
- added LED2, LED3, LED4, LED5, LED6, LED7, LED8, LED9: (no value), microbuilder:CHIPLED_0805
- added R14, R15, R16, R17, R18, R19, R20, R21: 470, microbuilder:0603
- moved C3 107.9 mm to (33.5, 51.5), turned to 90 degrees
- moved C1 104.7 mm to (19.5, 7.00)
- moved C2 98.4 mm to (19.5, 26.0)
- moved X3 76.2 mm to (3.50, 31.0), turned to 270 degrees
- moved R2 73.9 mm to (19.5, 11.0)
- moved R1 72.9 mm to (19.5, 9.00)
- moved R4 71.9 mm to (19.5, 22.0)
- moved IC10 67.7 mm to (19.5, 16.5), turned to 90 degrees
- moved C10 67.3 mm to (10.2, 41.8), turned to 270 degrees
- moved R3 66.9 mm to (19.5, 24.0)
- moved SJ4 65.0 mm to (30.5, 63.0), flipped to the bottom
- moved SJ2 62.1 mm to (30.5, 57.0), flipped to the bottom
- moved PS1 61.2 mm to (4.05, 44.4), turned to 90 degrees
- moved SJ1 57.8 mm to (30.5, 60.0), flipped to the bottom
- moved R5 55.8 mm to (14.9, 51.6)
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Connections:
- removed net N$12: IC3.1, IC3.4
- removed net N$13: C6.1, IC3.2, IC3.5, R8.2
- removed net N$16: IC4.1, IC4.4
- removed net N$17: C7.1, IC4.2, IC4.5, R9.2
- removed net N$20: IC5.1, IC5.4
- removed net N$21: C8.1, IC5.2, IC5.5, R10.2
- removed net N$24: IC6.1, IC6.4
- removed net N$25: C9.1, IC6.2, IC6.5, R11.2
- removed net N$28: IC7.1, IC7.4
- removed net N$33: IC8.1, IC8.4
- removed net N$34: C12.1, IC8.2, IC8.5, R13.2
- removed net N$8: IC2.1, IC2.4
- removed net N$9: C5.1, IC2.2, IC2.5, R7.2
- new net +VIN_RFM: C10.1, JP1.2, PS1.2
- new net N$37: LED2.A, R14.1
- new net N$38: LED3.A, R15.1
- new net N$39: LED4.A, R16.1
- new net N$40: LED5.A, R17.1
- new net N$41: LED6.A, R18.1
- new net N$42: LED7.A, R19.1
- new net N$43: LED8.A, R20.1
- new net N$44: LED9.A, R21.1
- new net N$45: C6.1, IC3.2, IC3.5, Q3.3, R8.2
- new net N$46: C7.1, IC4.2, IC4.5, Q4.3, R9.2
- new net N$47: C12.1, IC8.2, IC8.5, Q8.3, R13.2
- new net N$49: C9.1, IC6.2, IC6.5, Q6.3, R11.2
- new net N$50: C8.1, IC5.2, IC5.5, Q5.3, R10.2
- net +5V: now also C13.1
- net C1: now also IC9.7, R14.2; no longer IC9.4
- net C2: now also IC9.6, R15.2; no longer IC9.5
- net C3: now also IC9.5, R16.2; no longer IC9.6
- net C4: now also IC9.4, R17.2; no longer IC9.7
- net C5: now also IC9.12, R18.2; no longer IC9.9
- net C6: now also IC9.11, R19.2; no longer IC9.10
- net C7: now also IC9.10, R20.2; no longer IC9.11
- net C8: now also IC9.9, R21.2; no longer IC9.12
- net GND: now also C13.2, LED2.C, LED3.C, LED4.C, LED5.C, LED6.C, LED7.C, LED8.C, LED9.C
- net N$1: now also C4.1, IC1.2, IC1.5, Q1.3, R6.2; no longer IC1.1, IC1.4
- net N$11: now also IC2.1, IC2.4; no longer Q2.3
- net N$15: now also IC3.1, IC3.4; no longer Q3.3
- net N$19: now also IC4.1, IC4.4; no longer Q4.3
- net N$2: now also C4.2, IC1.1, IC1.4, R6.1; no longer C4.1, IC1.2, IC1.5, R6.2
- net N$23: now also IC5.1, IC5.4; no longer Q5.3
- net N$27: now also IC6.1, IC6.4; no longer Q6.3
- net N$29: now also Q7.3
- net N$3: now also C5.1, IC2.2, IC2.5, Q2.3, R7.2; no longer C4.2, Q1.3, R6.1
- net N$32: now also IC7.1, IC7.4; no longer Q7.3
- net N$36: now also IC8.1, IC8.4; no longer Q8.3
- net VCC_IN: no longer C10.1, JP1.2, PS1.2
Routing:
- net EP: track 0.00 -> 161.0 mm, vias 0 -> 8
- net +5V: track 0.00 -> 85.2 mm, vias 0 -> 2
- net VCC_IN: track 0.00 -> 54.2 mm, vias 0 -> 2
- net C8: track 0.00 -> 52.8 mm
- net C1: track 0.00 -> 50.0 mm
- net C7: track 0.00 -> 40.6 mm
- net C2: track 0.00 -> 37.6 mm
- net SDA: track 0.00 -> 36.4 mm, vias 0 -> 4
- net SCL: track 0.00 -> 35.4 mm, vias 0 -> 2
- net C6: track 0.00 -> 28.3 mm
- net SDA_IN: track 0.00 -> 27.4 mm
- net C3: track 0.00 -> 25.3 mm
- net SCL_IN: track 0.00 -> 25.2 mm
- net +VIN_RFM: track 0.00 -> 22.8 mm
- net N$46: track 0.00 -> 19.5 mm
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- added copper zone on layer 1, net GND
- added copper zone on layer 16, net GND
- added copper zone on layer 1, net GND_IN
- added copper zone on layer 16, net GND_IN
Other:
- board size 100 x 100 mm -> 60 x 100 mm
- board text added: "+3V3"
- board text added: "+5V"
- board text added: "B1"
- board text added: "B2"
- board text added: "B3"
- board text added: "B4"
- board text added: "B5"
- board text added: "B6"
- board text added: "B7"
- board text added: "B8"
- board text added: "DRAMCO"
- board text added: "GND"
- board text added: "Jarne Van Mulders"
- board text added: "Multiplexer V1.0"
- board text added: "Postdoctoral researcher"
- board text added: "Power"
- board text added: "SCL"
- board text added: "SDA"
