File: hardware/multiplexer-1vX/design.sch (EAGLE design)
At the start: 64 parts, among them IC10 ISO1540D, IC9 TCA9554APWR, X1 DG3XX-02-5.0, X10 DG3XX-02-5.0, X11 DG3XX-02-5.0, X2 04-JST-B4B-XH-A, X3 DG3XX-02-5.0, X4 DG3XX-02-5.0, X5 DG3XX-02-5.0, X6 DG3XX-02-5.0, X7 DG3XX-02-5.0, X8 DG3XX-02-5.0, X9 DG3XX-02-5.0

Commit message: Update hardware
Parts:
- added C13: (no value), microbuilder:CAP_CERAMIC0805
- added LED2, LED3, LED4, LED5, LED6, LED7, LED8, LED9: (no value), microbuilder:LED0805
- added R14, R15, R16, R17, R18, R19, R20, R21: 470, microbuilder:RESISTOR0603
Connections:
- removed net N$12: IC3.S1, IC3.S2
- removed net N$13: C6.P$1, IC3.G1, IC3.G2, R8.2
- removed net N$16: IC4.S1, IC4.S2
- removed net N$17: C7.P$1, IC4.G1, IC4.G2, R9.2
- removed net N$20: IC5.S1, IC5.S2
- removed net N$21: C8.P$1, IC5.G1, IC5.G2, R10.2
- removed net N$24: IC6.S1, IC6.S2
- removed net N$25: C9.P$1, IC6.G1, IC6.G2, R11.2
- removed net N$28: IC7.S1, IC7.S2
- removed net N$33: IC8.S1, IC8.S2
- removed net N$34: C12.P$1, IC8.G1, IC8.G2, R13.2
- removed net N$8: IC2.S1, IC2.S2
- removed net N$9: C5.P$1, IC2.G1, IC2.G2, R7.2
- new net +VIN_RFM: C10.P$1, JP1.2, PS1.+VIN
- new net N$37: LED2.A, R14.1
- new net N$38: LED3.A, R15.1
- new net N$39: LED4.A, R16.1
- new net N$40: LED5.A, R17.1
- new net N$41: LED6.A, R18.1
- new net N$42: LED7.A, R19.1
- new net N$43: LED8.A, R20.1
- new net N$44: LED9.A, R21.1
- new net N$45: C6.P$1, IC3.G1, IC3.G2, Q3.D, R8.2
- new net N$46: C7.P$1, IC4.G1, IC4.G2, Q4.D, R9.2
- new net N$47: C12.P$1, IC8.G1, IC8.G2, Q8.D, R13.2
- new net N$49: C9.P$1, IC6.G1, IC6.G2, Q6.D, R11.2
- new net N$50: C8.P$1, IC5.G1, IC5.G2, Q5.D, R10.2
- net +5V: now also C13.P$1
- net C1: now also IC9.P3, R14.2; no longer IC9.P0
- net C2: now also IC9.P2, R15.2; no longer IC9.P1
- net C3: now also IC9.P1, R16.2; no longer IC9.P2
- net C4: now also IC9.P0, R17.2; no longer IC9.P3
- net C5: now also IC9.P7, R18.2; no longer IC9.P4
- net C6: now also IC9.P6, R19.2; no longer IC9.P5
- net C7: now also IC9.P5, R20.2; no longer IC9.P6
- net C8: now also IC9.P4, R21.2; no longer IC9.P7
- net GND: now also C13.P$2, LED2.C, LED3.C, LED4.C, LED5.C, LED6.C, LED7.C, LED8.C, LED9.C
- net N$1: now also C4.P$1, IC1.G1, IC1.G2, Q1.D, R6.2; no longer IC1.S1, IC1.S2
- net N$11: now also IC2.S1, IC2.S2; no longer Q2.D
- net N$15: now also IC3.S1, IC3.S2; no longer Q3.D
- net N$19: now also IC4.S1, IC4.S2; no longer Q4.D
- net N$2: now also C4.P$2, IC1.S1, IC1.S2, R6.1; no longer C4.P$1, IC1.G1, IC1.G2, R6.2
- net N$23: now also IC5.S1, IC5.S2; no longer Q5.D
- net N$27: now also IC6.S1, IC6.S2; no longer Q6.D
- net N$29: now also Q7.D
- net N$3: now also C5.P$1, IC2.G1, IC2.G2, Q2.D, R7.2; no longer C4.P$2, Q1.D, R6.1
- net N$32: now also IC7.S1, IC7.S2; no longer Q7.D
- net N$36: now also IC8.S1, IC8.S2; no longer Q8.D
- net VCC_IN: no longer C10.P$1, JP1.2, PS1.+VIN
